File: PCB_Related.kicad_sch (KiCad schematic)
At the start: 0 parts

Commit message: Finished the schematics and assigning footprints
Parts:
- added C1: 1µF, Capacitor_SMD:C_0805_2012Metric, symbol Device:C_Small
- added C2, C3, C4, C5: 0.1µF, Capacitor_SMD:C_0805_2012Metric, symbol Device:C_Small
- added C6, C7: 22pF, Capacitor_SMD:C_0805_2012Metric, symbol Device:C_Small
- added D1, D2, D3, D4: SOD-123, Diode_SMD:D_SOD-123, symbol Device:D_Small
- added F1: 500mA, Fuse:Fuse_1206_3216Metric, symbol Device:Polyfuse_Small
- added MX1, MX2, MX3, MX4: MX-NoLED, MX_Alps_Hybrid:MX-10U-NoLED, symbol MX_Alps_Hybrid:MX-NoLED
- added R1, R2: 22, Resistor_SMD:R_0805_2012Metric, symbol Device:R_Small
- added R3, R4: 10K, Resistor_SMD:R_0805_2012Metric, symbol Device:R_Small
- added SW1: SW_Push, random-keyboard-parts:SKQG-1155865, symbol Switch:SW_Push
- added U1: ATmega32U4RC-A, Package_QFP:TQFP-44_10x10mm_P0.8mm, symbol MCU_Microchip_ATmega:ATmega32U4RC-A
- added USB1: Molex-0548190589, random-keyboard-parts:PJ-3200B-4A-Assembly, symbol random-keyboard-parts:Molex-0548190589
- added Y1: 16MHz, Crystal:Crystal_SMD_3225-4Pin_3.2x2.5mm, symbol Device:Crystal_GND24_Small
Connections:
- new net: C1.1, U1.6 (UCAP)
- new net: R4.1, SW1.2, U1.13 (~{RESET})
- new net: D4.2 (A), MX4.2 (ROW)
- new net: F1.1, USB1.5 (VBUS)
- new net: D2.2 (A), MX2.2 (ROW)
- new net: R2.2, U1.3 (D-)
- new net: C6.2, U1.16 (XTAL2), Y1.1
- new net: C7.2, U1.17 (XTAL1), Y1.3
- new net: R3.1, U1.33 (~{HWB}/PE2)
- new net: R1.2, U1.4 (D+)
- new net: D3.2 (A), MX3.2 (ROW)
- new net: D1.2 (A), MX1.2 (ROW)
- new net +5V: C2.1, C3.1, C4.1, C5.1, F1.2, R4.2, U1.14 (VCC), U1.2 (UVCC), U1.24 (AVCC), U1.34 (VCC), U1.44 (AVCC), U1.7 (VBUS)
- new net COL0: MX1.1 (COL), MX3.1 (COL), U1.37 (PF6)
- new net COL1: MX2.1 (COL), MX4.1 (COL), U1.36 (PF7)
- new net D+: R1.1, USB1.3 (D+)
- new net D-: R2.1, USB1.4 (D-)
- new net GND: C1.2, C2.2, C3.2, C4.2, C5.2, C6.1, C7.1, R3.2, SW1.1, U1.15 (GND), U1.23 (GND), U1.35 (GND), U1.43 (GND), U1.5 (UGND), USB1.1 (GND), USB1.6 (SHIELD), Y1.2, Y1.4
- new net ROW0: D1.1 (K), D2.1 (K), U1.39 (PF4)
- new net ROW1: D3.1 (K), D4.1 (K), U1.38 (PF5)
- no-connect marks 0 -> 1

Commit message: Finished the pcb and gerbers
Parts:
- added C8, C9: 0.1µF, Capacitor_SMD:C_0805_2012Metric, symbol Device:C_Small
- MX1, MX2, MX3, MX4: footprint MX_Alps_Hybrid:MX-10U-NoLED -> MX_Alps_Hybrid:MX-1U-NoLED
- USB1: footprint random-keyboard-parts:PJ-3200B-4A-Assembly -> random-keyboard-parts:Molex-0548190589
Connections:
- net +5V: now also C8.1, C9.1
- net COL0: now also U1.30 (PB6); no longer U1.37 (PF6)
- net COL1: now also U1.27 (PD7); no longer U1.36 (PF7)
- net GND: now also C8.2, C9.2
- net ROW0: now also U1.28 (PB4); no longer U1.39 (PF4)
- net ROW1: now also U1.29 (PB5); no longer U1.38 (PF5)
- net VCC: now reaches F1.1, USB1.5 (VBUS)
- no-connect marks 1 -> 2
