File: _autosave-PCB_Related.kicad_sch (KiCad schematic)
At the start: 13 parts, among them SW1 RotaryEncoder_Switch, U1 SK6812MINI-E, U2 SK6812MINI-E, U4 MOUDLE-SEEEDUINO-XIAO

Commit message: Added pictures and finished cad
Parts:
- removed D1, D2, D3, D4, D5: 1N4148, Diode_THT:D_DO-35_SOD27_P7.62mm_Horizontal, symbol 1N4148:1N4148
- removed U1, U2: SK6812MINI-E, SK6812MINI-E:SK6812MINI-E, symbol SK6812MINI-E:SK6812MINI-E
- added D1, D2, D3, D4, D5: D_Small, Diode_THT:D_DO-35_SOD27_P7.62mm_Horizontal, symbol Device:D_Small
- added D8, D9: SK6812-E, SK6812-E:LED_SK6812-E, symbol SK6812-E:SK6812-E
- added H2, H3, H4: MountingHole, MountingHole:MountingHole_3.7mm, symbol Mechanical:MountingHole
Connections:
- net A: now also D5.2 (A)
- net AUP: now also U4.5 (PA8_A4_D4_SDA)
- net B: now also U4.4 (PA11_A3_D3)
- net BDOWN: now also U4.6 (PA9_A5_D5_SCL)
- net GND: now also D8.3 (GND), D9.3 (GND)
- net LED: now also U4.7 (PB08_A6_D6_TX), D8.4 (DIN)
- net ROW0: now also D1.1 (K), D2.1 (K), D5.1 (K)
- net ROW1: now also D3.1 (K), D4.1 (K)
- net VCC: now also D8.1 (VDD), D9.1 (VDD)
- net at S3.1: now also D3.2 (A)
- net at S2.1: now also D2.2 (A)
- net at S4.1: now also D4.2 (A)
- net at S1.1: now also D1.2 (A)
- new net: D8.2 (DOUT), D9.4 (DIN)
- no-connect marks 8 -> 5
