File: PCB/PCB_Related.kicad_sch (KiCad schematic)
At the start: 46 parts, among them J1 USB4105-GF-A, Q1 L8050QLT1G, Q2 L8050QLT1G, SW1 SW_Push, SW2 SW_Push, U1 ESP32-C3-WROOM-02U-N4, U2 CP2102N-A02-GQFN28R, U3 AMS1117-3.3

Commit message: Updated Firmware and Production
Parts:
- removed C1, C2: 22pF, Capacitor_SMD:C_0805_2012Metric, symbol Device:C_Small
- removed C10, C11, C13, C6, C9: 0.1µF/50V, Capacitor_SMD:C_0805_2012Metric, symbol Device:C_Small
- removed C12, C14, C3, C7: 10µF/25V, Capacitor_SMD:C_0805_2012Metric, symbol Device:C_Small
- removed C4, C8: 1µF/16V, Capacitor_SMD:C_0805_2012Metric, symbol Device:C_Small
- removed D10, D6, D8, D9: Z1N5819HW-7-F, Diode_SMD:D_SOD-123, symbol Device:D_Small
- removed D3: LESD5D5.0CT1G, Diode_SMD:D_SOD-123, symbol Device:D_Small
- removed H1, H2, H3, H4: MountingHole, MountingHole:MountingHole_3.2mm_M3, symbol Mechanical:MountingHole
- removed J1: USB4105-GF-A, USB4105-GF-A:GCT_USB4105-GF-A, symbol USB4105-GF-A:USB4105-GF-A
- removed Q1, Q2: L8050QLT1G, SMD-TRANSISTORS-NPN-25V-500MW_SOT-23_:SOT-23, symbol SMD-TRANSISTORS-NPN-25V-500MW_SOT-23_:SMD-TRANSISTORS-NPN-25V-500MW_SOT-23_
- removed R1, R2: 51k, Resistor_SMD:R_0805_2012Metric, symbol Device:R_Small
- removed R10: 1K, Resistor_SMD:R_0805_2012Metric, symbol Device:R_Small
- removed R11: 22.1K, Resistor_SMD:R_0805_2012Metric, symbol Device:R_Small
- removed R12: 47.5K, Resistor_SMD:R_0805_2012Metric, symbol Device:R_Small
- removed R13, R14, R7, R8: 0, Resistor_SMD:R_0805_2012Metric, symbol Device:R_Small
- removed R15, R16, R9: 10K, Resistor_SMD:R_0805_2012Metric, symbol Device:R_Small
- removed SW1, SW2: SW_Push, random-keyboard-parts:SKQG-1155865, symbol Switch:SW_Push
- removed U1: ESP32-C3-WROOM-02U-N4, ESP32-C3-WROOM-02U-N4:XCVR_ESP32-C3-WROOM-02U-N4, symbol ESP32-C3-WROOM-02U-N4:ESP32-C3-WROOM-02U-N4
- removed U2: CP2102N-A02-GQFN28R, CP2102N-A02-GQFN28R:IC_CP2102N-A02-GQFN28R, symbol CP2102N-A02-GQFN28R:CP2102N-A02-GQFN28R
- removed U3: AMS1117-3.3, AMS1117-3.3:SOT229P700X180-4N, symbol AMS1117-3.3:AMS1117-3.3
- added D1, D2, D3, D4: 1N4148, 1N4148:DO35-7, symbol 1N4148:1N4148
- added U4: MOUDLE-SEEEDUINO-XIAO, XIAO_RP2040:XIAO-Generic-Hybrid-14P-2.54-21X17.8MM, symbol XIAO_RP2040:MOUDLE-SEEEDUINO-XIAO
Connections:
- net COL0: now also U4.11 (PA6_A10_D10_MOSI)
- net COL1: now also U4.10 (PA5_A9_D9_MISO)
- net GND: now also U4.13 (GND)
- net ROW0: now also D1.C, D2.C, U4.9 (PA7_A8_D8_SCK)
- net ROW1: now also D3.C, D4.C, U4.8 (PB09_A7_D7_RX)
- net at S3.1: now also D4.A
- net at S4.1: now also D3.A
- net at S1.1: now also D1.A
- net at S2.1: now also D2.A
- no-connect marks 24 -> 9
